File: Zamek_RFID_Hardware/Zamek_RFID_Hardware/Zamek_RFID_Hardware.kicad_pcb (KiCad board)
At the start: 2 copper layers, 72 x 57.2 mm, 30 parts, among them J1 Conn_01x08, J2 Conn_01x08, J3 Conn_01x04, J4 Conn_01x03, Q1 BC547

Commit message: hw: set R2 to 300 ohm, tidy up schematic labels and title block
Parts:
- R2: value 200 -> 300
Changed lines of the file:
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@@
 			)
 		)
-		(property "Value" "200"
+		(property "Value" "300"
 			(at 5.08 2.37 270)
 			(layer "F.Fab")
